Commit message: 1. Add USD file for PushMazeA-3D 2. Fix the error in set_goal functions of PushT tasks

File: tasks/pushmaze_3d/assets/robot/urdf/ur5e_probe_mazeA.urdf (robot description, URDF)
Before this commit: robot ur5e, 19 links, 18 joints
Links:
- link obs_L1_1: geometry collision box size=0.07 0.01 0.05; visual box size=0.07 0.01 0.05
- link obs_L1_2: geometry collision box size=0.01 0.07 0.05; visual box size=0.01 0.07 0.05
- link obs_L2_1: geometry collision box size=0.07 0.01 0.05; visual box size=0.07 0.01 0.05
- link obs_L2_2: geometry collision box size=0.01 0.07 0.05; visual box size=0.01 0.07 0.05
- link obs_L3_1: geometry collision box size=0.07 0.01 0.05; visual box size=0.07 0.01 0.05
- link obs_L3_2: geometry collision box size=0.01 0.07 0.05; visual box size=0.01 0.07 0.05
- link obs_L4_1: geometry collision box size=0.07 0.01 0.05; visual box size=0.07 0.01 0.05
- link obs_L4_2: geometry collision box size=0.01 0.07 0.05; visual box size=0.01 0.07 0.05
- link table: geometry collision box size=0.5 0.5 0.3; visual box size=0.5 0.5 0.3
Joints:
- joint base_link_ground: origin xyz=-0.7 0.0 0 rpy=0 0 0 -> xyz=-0.5 0.0 0 rpy=0 0 0
- joint obs_L1_1: origin xyz=0.6 0.3 0 rpy=0 0 0 -> xyz=0.06 0.03 0.15 rpy=0 0 0
- joint obs_L1_2: origin xyz=0.3 0.6 0 rpy=0 0 0 -> xyz=0.03 0.06 0.15 rpy=0 0 0
- joint obs_L2_1: origin xyz=-0.6 -0.3 0 rpy=0 0 0 -> xyz=-0.06 -0.03 0.15 rpy=0 0 0
- joint obs_L2_2: origin xyz=-0.3 -0.6 0 rpy=0 0 0 -> xyz=-0.03 -0.06 0.15 rpy=0 0 0
- joint obs_L3_1: origin xyz=0.6 -0.3 0 rpy=0 0 0 -> xyz=0.06 -0.03 0.15 rpy=0 0 0
- joint obs_L3_2: origin xyz=0.3 -0.6 0 rpy=0 0 0 -> xyz=0.03 -0.06 0.15 rpy=0 0 0
- joint obs_L4_1: origin xyz=-0.6 0.3 0 rpy=0 0 0 -> xyz=-0.06 0.03 0.15 rpy=0 0 0
- joint obs_L4_2: origin xyz=-0.3 0.6 0 rpy=0 0 0 -> xyz=-0.03 0.06 0.15 rpy=0 0 0
- joint table_ground: origin xyz=0.0 0.0 0 rpy=0 0 0 -> xyz=0.0 0.0 0.15 rpy=0 0 0
